File: MMA7361/acel.sch (KiCad schematic (older format))
At the start: 13 parts, among them J1 Conn_01x05, J2 Conn_01x05, U1 RT9701, U2 MMA7260Q

Commit message: The Schematic have been fixed
Parts:
- U2: footprint MMA7260Q:QFN-16 -> QFN-16
Connections:
- net labels added: SelfTest
- net labels removed: X, Y, Z
- wire segments 48 -> 52
- no-connect marks 2 -> 1

Commit message: More changes
Parts:
- U2: footprint QFN-16 -> MMA7260Q:QFN-16
Changed lines of the file:
@@
 F 0 "U2" H 9150 3567 50  0000 C CNN
 F 1 "MMA7260Q" H 9150 3476 50  0000 C CNN
-F 2 "QFN-16" H 9250 3450 50  0001 L BNN
+F 2 "MMA7260Q:QFN-16" H 9250 3450 50  0001 L BNN
 F 3 "NXP Semiconductors" H 9700 3300 50  0001 L BNN
 F 4 "MMA7260Q" H 9650 2050 50  0001 L BNN "Field5"

Commit message: the files have been fixed
Parts:
- added F1, F2, F3: Fiducial, Fiducial:Fiducial_0.5mm_Dia_1mm_Outer, symbol Mechanical:MountingHole
- U1: value RT9701 -> RT9161
- U2: value MMA7260Q -> MMA7361L
Connections:
- net labels added: Fiducial, U1_RT9701, U2_MMA7361L
- wire segments 52 -> 51

Commit message: The last version have been added
Parts:
- C1, C3, C4, C5, C7: symbol Device:C -> MMA7361-rescue:C-Device
- C2, C6: symbol Device:CP1 -> MMA7361-rescue:CP1-Device
- D1: symbol Device:LED -> MMA7361-rescue:LED-Device
- F1, F2, F3: symbol Mechanical:MountingHole -> MMA7361-rescue:MountingHole-Mechanical
- J1, J2: symbol Connector_Generic:Conn_01x05 -> MMA7361-rescue:Conn_01x05-Connector_Generic
- R1: symbol Device:R -> MMA7361-rescue:R-Device
- U1: symbol Power_Management:RT9701 -> MMA7361-rescue:RT9701-Power_Management
Changed lines of the file:
@@
 EESchema Schematic File Version 4
+LIBS:MMA7361-cache
 EELAYER 26 0
 EELAYER END
@@
 $EndDescr
 $Comp
-L Device:C C4
+L MMA7361-rescue:C-Device C4
 U 1 1 5BC120D2
 P 3000 2750
@@
 $EndComp
 $Comp
-L Device:CP1 C2
+L MMA7361-rescue:CP1-Device C2
 U 1 1 5BC123C9
 P 2300 2750
@@
 $EndComp
 $Comp
-L Power_Management:RT9701 U1
+L MMA7361-rescue:RT9701-Power_Management U1
 U 1 1 5BC26997
 P 3950 2700
@@
 $EndComp
 $Comp
-L Device:CP1 C6
+L MMA7361-rescue:CP1-Device C6
 U 1 1 5BC26B05
 P 5000 2750
@@
 $EndComp
 $Comp
-L power:GND #PWR03
+L MMA7361-rescue:GND-power #PWR03
 U 1 1 5BC26BFC
 P 3950 3050
@@
 $EndComp
 $Comp
-L Device:C C1
+L MMA7361-rescue:C-Device C1
 U 1 1 5BC2906F
 P 7500 2650
@@
 $EndComp
 $Comp
-L Device:C C3
+L MMA7361-rescue:C-Device C3
 U 1 1 5BC2913B
 P 6550 2350
@@
 $EndComp
 $Comp
-L Device:C C5
+L MMA7361-rescue:C-Device C5
 U 1 1 5BC292F0
 P 7000 2500
@@
 $EndComp
 $Comp
-L Device:LED D1
+L MMA7361-rescue:LED-Device D1
 U 1 1 5BC2963F
 P 10850 3750
@@
 $EndComp
 $Comp
-L power:GND #PWR04
+L MMA7361-rescue:GND-power #PWR04
 U 1 1 5BC29FE3
 P 10850 4700
@@
 $EndComp
 $Comp
-L Device:R R1
+L MMA7361-rescue:R-Device R1
 U 1 1 5BC2A087
 P 10850 2600
@@
 	3950 2900 5000 2900
 $Comp
-L power:GND #PWR02
+L MMA7361-rescue:GND-power #PWR02
 U 1 1 5BC2D65B
 P 6300 3250
@@
 $EndComp
 $Comp
-L Device:C C7
+L MMA7361-rescue:C-Device C7
 U 1 1 5BC2F1C2
 P 7950 2950
@@
 Connection ~ 4450 2600
 $Comp
-L power:PWR_FLAG #FLG0101
+L MMA7361-rescue:PWR_FLAG-power #FLG0101
 U 1 1 5BC4F7C2
 P 4450 3050
@@
 Connection ~ 3950 3050
 $Comp
-L Connector_Generic:Conn_01x05 J1
+L MMA7361-rescue:Conn_01x05-Connector_Generic J1
 U 1 1 5BC514EF
 P 8850 4600
+AR Path="/5BC514EF" Ref="J1"  Part="1"
+AR Path="/5BC12037/5BC514EF" Ref="J1"  Part="1"
 F 0 "J1" H 8930 4642 50  0000 L CNN
 F 1 "Conn_01x05" H 8930 4551 50  0001 L CNN
@@
 $EndComp
 $Comp
-L Connector_Generic:Conn_01x05 J2
+L MMA7361-rescue:Conn_01x05-Connector_Generic J2
 U 1 1 5BC52AEF
 P 5750 2600
+AR Path="/5BC52AEF" Ref="J2"  Part="1"
+AR Path="/5BC12037/5BC52AEF" Ref="J2"  Part="1"
 F 0 "J2" H 5829 2596 50  0000 L CNN
 F 1 "Conn_01x05" H 5830 2551 50  0001 L CNN
@@
 Connection ~ 2300 2600
 $Comp
-L power:+5V #PWR0101
+L MMA7361-rescue:+5V-power #PWR0101
 U 1 1 5BC5B9BB
 P 1450 2600
@@
 $EndComp
 $Comp
-L power:PWR_FLAG #FLG0102
+L MMA7361-rescue:PWR_FLAG-power #FLG0102
 U 1 1 5BC6426B
 P 800 2600
@@
 $EndComp
 $Comp
-L power:VCC #PWR0102
+L MMA7361-rescue:VCC-power #PWR0102
 U 1 1 5BCC985E
 P 8300 2950
@@
 	9750 2250 10150 2250
 $Comp
-L power:VCC #PWR0103
+L MMA7361-rescue:VCC-power #PWR0103
 U 1 1 5BCDE47F
 P 5000 2450
@@
 Connection ~ 5000 2600
 $Comp
-L power:VCC #PWR0104
+L MMA7361-rescue:VCC-power #PWR0104
 U 1 1 5BD65502
 P 10850 1700
@@
 	8300 2950 8550 2950
 $Comp
-L Mechanical:MountingHole F1
+L MMA7361-rescue:MountingHole-Mechanical F1
 U 1 1 5BDB6852
 P 1750 6450
@@
 $EndComp
 $Comp
-L Mechanical:MountingHole F2
+L MMA7361-rescue:MountingHole-Mechanical F2
 U 1 1 5BDB6900
 P 1750 6950
@@
 $EndComp
 $Comp
-L Mechanical:MountingHole F3
+L MMA7361-rescue:MountingHole-Mechanical F3
 U 1 1 5BDB69CF
 P 3100 6450
