File: MMA7361/MMA7361.kicad_pcb (KiCad board)
At the start: 2 copper layers, 23.4 x 22.9 mm, 13 parts, among them J1 Conn_01x05, J2 Conn_01x05, U1 RT9701, U2 MMA7260Q

Commit message: More changes
Parts:
- moved J2 13.4 mm to (150.2, 92.8)
- moved U2 7.31 mm to (142.9, 94.6)
- moved C2 6.74 mm to (147.9, 89.2)
- moved C6 6.51 mm to (147.4, 85.5)
- moved C4 6.04 mm to (134.9, 85.4)
- moved C5 6.04 mm to (134.7, 97.8)
- moved C1 6.04 mm to (134.6, 89.2)
- moved C3 6.04 mm to (134.7, 93.3)
- moved U1 5.85 mm to (141.2, 86.8)
- moved C7 5.70 mm to (140.7, 100.7)
- moved D1 5.70 mm to (145.3, 100.7)
- moved R1 5.70 mm to (149.6, 100.7)
- moved J1 5.43 mm to (133.3, 100.6)
Connections:
- C1 pad 2: /MMA 7361 Module/X -> Net-(C1-Pad2)
- C3 pad 2: /MMA 7361 Module/Y -> Net-(C3-Pad2)
- C5 pad 2: /MMA 7361 Module/Z -> Net-(C5-Pad2)
- C6 pad 1: /MMA 7361 Module/VCC -> VCC
- C7 pad 1: GND -> VCC
- C7 pad 2: /MMA 7361 Module/VCC -> GND
- J1 pad 2: /MMA 7361 Module/VCC -> VCC
- J1 pad 5: Net-(J1-Pad5) -> /MMA 7361 Module/SelfTest
- J2 pad 1: /MMA 7361 Module/X -> GND
- J2 pad 2: /MMA 7361 Module/Y -> GND
- J2 pad 3: /MMA 7361 Module/Z -> GND
- R1 pad 2: /MMA 7361 Module/VCC -> VCC
- U1 pad 1: /MMA 7361 Module/VCC -> VCC
- U1 pad 5: /MMA 7361 Module/VCC -> VCC
- U2 pad 1: /MMA 7361 Module/Og-Detect -> Net-(U2-Pad1)
- U2 pad 10: (no net) -> /MMA 7361 Module/g-Select
- U2 pad 11: (no net) -> Net-(U2-Pad11)
- U2 pad 12: /MMA 7361 Module/Sleep -> Net-(U2-Pad12)
- U2 pad 13: /MMA 7361 Module/Z -> /MMA 7361 Module/SelfTest
- U2 pad 14: /MMA 7361 Module/Y -> (no net)
- U2 pad 15: /MMA 7361 Module/X -> (no net)
- U2 pad 2: /MMA 7361 Module/g-Select -> Net-(C3-Pad2)
- U2 pad 3: /MMA 7361 Module/VCC -> Net-(C5-Pad2)
- U2 pad 4: GND -> Net-(C1-Pad2)
- U2 pad 5: (no net) -> GND
- U2 pad 6: (no net) -> VCC
- U2 pad 7: (no net) -> /MMA 7361 Module/Sleep
- U2 pad 8: (no net) -> Net-(U2-Pad8)
- U2 pad 9: (no net) -> /MMA 7361 Module/Og-Detect
Routing:
- net /MMA 7361 Module/VCC: track 6.06 -> 0.00 mm
- net VCC: track 0.00 -> 6.06 mm
- net Net-(C5-Pad2): track 0.00 -> 4.49 mm
- net /MMA 7361 Module/Z: track 4.49 -> 0.00 mm
- added copper zone on F.Cu, net GND
Other:
- board size 23.4 x 22.9 mm -> 24.1 x 24.3 mm
- net class Default: clearance 0.8 -> 0.25; trace_width 0.2 -> 0.25; via_drill 0.6 -> 0.5
- net class Test removed
- rule trace_clearance: 0.8 -> 0.25
- rule trace_min: 0.2 -> 0.25
- rule via_min_drill: 0.3 -> 0.5
- rule via_min_size: 0.4 -> 1

Commit message: The last change have been added
Parts:
- moved C1 25.3 mm to (158.8, 96.8), turned to 180 degrees
- moved D1 19.4 mm to (162.3, 91.4), turned to 90 degrees
- moved C7 19.1 mm to (158.7, 94.2)
- moved C5 19.1 mm to (153.7, 96.8), turned to 180 degrees
- moved R1 19.0 mm to (161.5, 85.9), turned to 90 degrees
- moved U1 15.9 mm to (157.1, 85.5)
- moved J1 15.7 mm to (147.3, 93.5), turned to 180 degrees
- moved C3 15.1 mm to (149.3, 96.8), turned to 180 degrees
- moved C4 14.0 mm to (148.8, 85.6), turned to 90 degrees
- moved J2 13.2 mm to (155.7, 80.8), turned to 270 degrees
- moved C6 12.8 mm to (159.3, 90.4)
- moved U2 10.7 mm to (153.2, 91.7)
- moved C2 5.37 mm to (151.9, 85.6), turned to 90 degrees
Routing:
- net GND: track 0.00 -> 33.2 mm
- net VCC: track 6.06 -> 37.8 mm, vias 0 -> 2
- net /MMA 7361 Module/Sleep: track 0.00 -> 13.7 mm, vias 0 -> 2
- net /MMA 7361 Module/g-Select: track 0.00 -> 11.0 mm
- net /MMA 7361 Module/Og-Detect: track 0.00 -> 9.40 mm, vias 0 -> 2
- net Net-(C3-Pad2): track 0.00 -> 7.40 mm
- net Net-(C1-Pad2): track 0.00 -> 4.04 mm
- net Net-(D1-Pad2): track 0.00 -> 3.84 mm
- net /MMA 7361 Module/SelfTest: track 0.00 -> 3.39 mm
- net Net-(C5-Pad2): track 4.49 -> 2.75 mm
- net +5V: track 10.9 -> 9.63 mm
Other:
- board size 24.1 x 24.3 mm -> 22.4 x 20.3 mm
- rule pad_to_mask_clearance: 0 -> 0.2
- rule trace_min: 0.25 -> 0.2
- rule via_min_drill: 0.5 -> 0.3
- rule via_min_size: 1 -> 0.4
- board text added: "2"
- board text added: "2018"
- board text added: "MMA 7361"
- board text added: "[1 ]"

Commit message: the files have been fixed
Parts:
- added F1: Fiducial, Fiducial:Fiducial_0.5mm_Dia_1mm_Outer, F.Cu at (144.0, 97.0)
- added F2: Fiducial, Fiducial:Fiducial_0.5mm_Dia_1mm_Outer, F.Cu at (163.0, 81.0)
- added F3: Fiducial, Fiducial:Fiducial_0.5mm_Dia_1mm_Outer, F.Cu at (144.0, 81.0)
- U1: value RT9701 -> RT9161
- U2: value MMA7260Q -> MMA7361L
Other:
- board text added: "IND. ARG"
Changed lines of the file:
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@@
   (general
     (thickness 1.6)
-    (drawings 8)
+    (drawings 9)
     (tracks 86)
     (zones 0)
-    (modules 13)
+    (modules 16)
     (nets 17)
   )
   (page A4)
   (layers
-    (0 F.Cu signal)
-    (31 B.Cu signal)
+    (0 F.Cu mixed)
+    (31 B.Cu mixed)
     (32 B.Adhes user)
     (33 F.Adhes user)
@@
     (47 F.CrtYd user)
     (48 B.Fab user)
-    (49 F.Fab user hide)
+    (49 F.Fab user)
   )
   (setup
@@
     (pad_to_mask_clearance 0.2)
     (solder_mask_min_width 0.25)
-    (aux_axis_origin 0 0)
+    (aux_axis_origin 163 81)
+    (grid_origin 163 81)
     (visible_elements FFFDFF7F)
     (pcbplotparams
@@
     (add_net VCC)
   )
+  (module Fiducial:Fiducial_0.5mm_Dia_1mm_Outer (layer F.Cu)
+    (at 144 81)
+    (descr "Circular Fiducial, 0.5mm bare copper top; 1mm keepout (Level C)")
+    (tags marker)
+    (attr virtual)
+    (fp_text reference F3 (at 0 -1.5) (layer F.SilkS)
+      (effects (font (size 1 1) (thickness 0.15)))
+    )
+    (fp_text value Fiducial (at 0 1.5) (layer F.Fab)
+      (effects (font (size 1 1) (thickness 0.15)))
+    )
+    (fp_circle (center 0 0) (end 0.5 0) (layer F.Fab) (width 0.1))
+    (fp_text user %R (at 0 0) (layer F.Fab)
+      (effects (font (size 0.2 0.2) (thickness 0.04)))
+    )
+    (fp_circle (center 0 0) (end 0.75 0) (layer F.CrtYd) (width 0.05))
+    (pad ~ smd circle (at 0 0) (size 0.5 0.5) (layers F.Cu F.Mask)
+      (solder_mask_margin 0.25) (clearance 0.25))
+  )
+  (module Fiducial:Fiducial_0.5mm_Dia_1mm_Outer (layer F.Cu)
+    (at 163 81)
+    (descr "Circular Fiducial, 0.5mm bare copper top; 1mm keepout (Level C)")
+    (tags marker)
+    (attr virtual)
+    (fp_text reference F2 (at 0 -1.5) (layer F.SilkS)
+      (effects (font (size 1 1) (thickness 0.15)))
+    )
+    (fp_text value Fiducial (at 0 1.5) (layer F.Fab)
+      (effects (font (size 1 1) (thickness 0.15)))
+    )
+    (fp_circle (center 0 0) (end 0.75 0) (layer F.CrtYd) (width 0.05))
+    (fp_text user %R (at 0 0) (layer F.Fab)
+      (effects (font (size 0.2 0.2) (thickness 0.04)))
+    )
+    (fp_circle (center 0 0) (end 0.5 0) (layer F.Fab) (width 0.1))
+    (pad ~ smd circle (at 0 0) (size 0.5 0.5) (layers F.Cu F.Mask)
+      (solder_mask_margin 0.25) (clearance 0.25))
+  )
+  (module Fiducial:Fiducial_0.5mm_Dia_1mm_Outer (layer F.Cu)
+    (at 144 97)
+    (descr "Circular Fiducial, 0.5mm bare copper top; 1mm keepout (Level C)")
+    (tags marker)
+    (attr virtual)
+    (fp_text reference F1 (at 0 -1.5) (layer F.SilkS)
+      (effects (font (size 1 1) (thickness 0.15)))
+    )
+    (fp_text value Fiducial (at 0 1.5) (layer F.Fab)
+      (effects (font (size 1 1) (thickness 0.15)))
+    )
+    (fp_circle (center 0 0) (end 0.5 0) (layer F.Fab) (width 0.1))
+    (fp_text user %R (at 0 0) (layer F.Fab)
+      (effects (font (size 0.2 0.2) (thickness 0.04)))
+    )
+    (fp_circle (center 0 0) (end 0.75 0) (layer F.CrtYd) (width 0.05))
+    (pad ~ smd circle (at 0 0) (size 0.5 0.5) (layers F.Cu F.Mask)
+      (solder_mask_margin 0.25) (clearance 0.25))
+  )
   (module MMA7260Q:QFN-16 (layer F.Cu)
     (at 153.162 91.694)
@@
       (effects (font (size 0.801591 0.801591) (thickness 0.05)))
     )
-    (fp_text value MMA7260Q (at -0.2 -3.8) (layer F.SilkS)
+    (fp_text value MMA7361L (at -0.2 -3.8) (layer F.SilkS)
       (effects (font (size 0.800764 0.800764) (thickness 0.05)))
     )
@@
       (effects (font (size 1 1) (thickness 0.15)))
     )
-    (fp_text value RT9701 (at 0.218 2.64) (layer F.Fab)
+    (fp_text value RT9161 (at 0.218 2.64) (layer F.Fab)
       (effects (font (size 1 1) (thickness 0.15)))
     )
@@
     )
   )
+  (gr_text "IND. ARG" (at 145 86 90) (layer B.Cu)
+    (effects (font (size 1.2 1.2) (thickness 0.25)) (justify mirror))
+  )
+  (gr_text 2018 (at 147 85 90) (layer F.Cu)
+    (effects (font (size 1 1) (thickness 0.25)))
+  )
   (gr_text 2 (at 147.5 80) (layer B.Cu)
     (effects (font (size 1 1) (thickness 0.25)))
@@
   (gr_text "[1 ]" (at 147 80) (layer F.Cu)
     (effects (font (size 1 1) (thickness 0.25)))
-  )
-  (gr_text 2018 (at 147 85 90) (layer B.SilkS)
-    (effects (font (size 1 1) (thickness 0.2)) (justify mirror))
   )
   (gr_text "MMA\n7361" (at 160 81) (layer F.SilkS)
@@
   (gr_line (start 164.846 78.486) (end 164.846 98.806) (layer Edge.Cuts) (width 0.1))
   (gr_line (start 142.494 78.486) (end 164.846 78.486) (layer Edge.Cuts) (width 0.1))
-  (segment (start 161.544 89.644) (end 162.306 90.406) (width 0.8) (layer F.Cu) (net 1))
-  (segment (start 161.544 86.886) (end 161.544 89.644) (width 0.8) (layer F.Cu) (net 1))
+  (segment (start 161.544 89.644) (end 162.306 90.406) (width 0.5) (layer F.Cu) (net 1))
+  (segment (start 161.544 86.886) (end 161.544 89.644) (width 0.5) (layer F.Cu) (net 1))
   (segment (start 152.842 85.532) (end 151.892 84.582) (width 0.5) (layer F.Cu) (net 2))
   (segment (start 155.702 85.532) (end 152.842 85.532) (width 0.5) (layer F.Cu) (net 2))
@@
       )
     )
+  )
+  (zone (net 0) (net_name "") (layer B.Mask) (hatch edge 0.508)
+    (connect_pads (clearance 0.508))
+    (min_thickness 0.254)
+    (fill yes (arc_segments 16) (thermal_gap 0.508) (thermal_bridge_width 0.508))
+    (polygon
+      (pts
+        (xy 144 82) (xy 146 82) (xy 146 90) (xy 144 90)
+      )
+    )

Commit message: New changes have been added
Other:
- board text added: "* Componente: MMA7361 * Pista: 0.250 mm * Margen: 0.25 mm * Mínimo ancho pista: 0.2 mm * Mínimo tamaño vía: 0.4 mm * Minimum via diameter: 1 mm * Terminación: HASL"
- board text added: "NOTA: P1 no fue posible hallar el modelo 3d"
Changed lines of the file:
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@@
-(kicad_pcb (version 20171130) (host pcbnew 5.0.0-fee4fd1~66~ubuntu16.04.1)
+(kicad_pcb (version 20171130) (host pcbnew "(5.0.0)")
   (general
     (thickness 1.6)
-    (drawings 9)
+    (drawings 11)
     (tracks 86)
     (zones 0)
@@
     (aux_axis_origin 163 81)
     (grid_origin 163 81)
-    (visible_elements FFFDFF7F)
+    (visible_elements 7FFDFFFF)
     (pcbplotparams
       (layerselection 0x311fc_ffffffff)
@@
       (effects (font (size 0.801591 0.801591) (thickness 0.05)))
     )
-    (fp_text value MMA7361L (at -0.2 -3.8) (layer F.SilkS)
+    (fp_text value MMA7361L (at -0.2 -3.8) (layer F.Fab)
       (effects (font (size 0.800764 0.800764) (thickness 0.05)))
     )
@@
     )
   )
+  (gr_text "NOTA: P1 no fue posible hallar el modelo 3d" (at 187.93 98.29) (layer Dwgs.User)
+    (effects (font (size 1 1) (thickness 0.2)))
+  )
+  (gr_text "* Componente: MMA7361\n* Pista: 0.250 mm\n* Margen: 0.25 mm\n* Mínimo ancho pista: 0.2 mm\n* Mínimo tamaño vía: 0.4 mm\n* Minimum via diameter: 1 mm\n* Terminación: HASL" (at 186.51 82.3) (layer Dwgs.User)
+    (effects (font (size 1 1) (thickness 0.2)))
+  )
   (gr_text "IND. ARG" (at 145 86 90) (layer B.Cu)

Commit message: The last version have been added
Parts:
- U2: footprint MMA7260Q:QFN-16 -> qfn-16:QFN-16
Changed lines of the file:
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@@
-(kicad_pcb (version 20171130) (host pcbnew "(5.0.0)")
+(kicad_pcb (version 20171130) (host pcbnew "(5.0.1)-4")
   (general
     (thickness 1.6)
-    (drawings 11)
+    (drawings 13)
     (tracks 86)
     (zones 0)
@@
     (add_net VCC)
   )
+  (module qfn-16:QFN-16 (layer F.Cu)
+    (at 153.162 91.694)
+    (descr "16 LEAD QFN CASE 1622-01<br>E.g. MMA7260Q")
+    (attr smd)
+    (fp_text reference U2 (at -3.81 0) (layer F.SilkS)
+      (effects (font (size 0.801591 0.801591) (thickness 0.05)))
+    )
+    (fp_text value MMA7361L (at -0.2 -3.8) (layer F.Fab)
+      (effects (font (size 0.800764 0.800764) (thickness 0.05)))
+    )
+    (fp_circle (center -3.7 3.5) (end -3.2877 3.5) (layer F.SilkS) (width 0.1))
+    (fp_line (start 3 3) (end 3 2.5) (layer F.SilkS) (width 0.127))
+    (fp_line (start 2.5 3) (end 3 3) (layer F.SilkS) (width 0.127))
+    (fp_line (start -3 3) (end -2.5 3) (layer F.SilkS) (width 0.127))
+    (fp_line (start -3 2.5) (end -3 3) (layer F.SilkS) (width 0.127))
+    (fp_line (start 3 -3) (end 3 -2.5) (layer F.SilkS) (width 0.127))
+    (fp_line (start 2.5 -3) (end 3 -3) (layer F.SilkS) (width 0.127))
+    (fp_line (start -3 -3) (end -3 -2.5) (layer F.SilkS) (width 0.127))
+    (fp_line (start -2.5 -3) (end -3 -3) (layer F.SilkS) (width 0.127))
+    (fp_line (start -3 3) (end -3 -3) (layer F.CrtYd) (width 0.127))
+    (fp_line (start 3 3) (end -3 3) (layer F.CrtYd) (width 0.127))
+    (fp_line (start 3 -3) (end 3 3) (layer F.CrtYd) (width 0.127))
+    (fp_line (start -3 -3) (end 3 -3) (layer F.CrtYd) (width 0.127))
+    (pad 16 smd rect (at -2.75 1.5 270) (size 0.5 0.55) (layers F.Cu F.Paste F.Mask))
+    (pad 15 smd rect (at -2.75 0.5 270) (size 0.5 0.55) (layers F.Cu F.Paste F.Mask))
+    (pad 14 smd rect (at -2.75 -0.5 270) (size 0.5 0.55) (layers F.Cu F.Paste F.Mask))
+    (pad 13 smd rect (at -2.75 -1.5 270) (size 0.5 0.55) (layers F.Cu F.Paste F.Mask)
+      (net 12 "/MMA 7361 Module/SelfTest"))
+    (pad 12 smd rect (at -1.5 -2.75 180) (size 0.5 0.55) (layers F.Cu F.Paste F.Mask)
+      (net 16 "Net-(U2-Pad12)"))
+    (pad 11 smd rect (at -0.5 -2.75 180) (size 0.5 0.55) (layers F.Cu F.Paste F.Mask)
+      (net 15 "Net-(U2-Pad11)"))
+    (pad 10 smd rect (at 0.5 -2.75 180) (size 0.5 0.55) (layers F.Cu F.Paste F.Mask)
+      (net 5 "/MMA 7361 Module/g-Select"))
+    (pad 9 smd rect (at 1.5 -2.75 180) (size 0.5 0.55) (layers F.Cu F.Paste F.Mask)
+      (net 4 "/MMA 7361 Module/Og-Detect"))
+    (pad 8 smd rect (at 2.75 -1.5 90) (size 0.5 0.55) (layers F.Cu F.Paste F.Mask)
+      (net 14 "Net-(U2-Pad8)"))
+    (pad 7 smd rect (at 2.75 -0.5 90) (size 0.5 0.55) (layers F.Cu F.Paste F.Mask)
+      (net 6 "/MMA 7361 Module/Sleep"))
+    (pad 6 smd rect (at 2.75 0.5 90) (size 0.5 0.55) (layers F.Cu F.Paste F.Mask)
+      (net 11 VCC))
+    (pad 5 smd rect (at 2.75 1.5 90) (size 0.5 0.55) (layers F.Cu F.Paste F.Mask)
+      (net 2 GND))
+    (pad 4 smd rect (at 1.5 2.75) (size 0.5 0.55) (layers F.Cu F.Paste F.Mask)
+      (net 8 "Net-(C1-Pad2)"))
+    (pad 3 smd rect (at 0.5 2.75) (size 0.5 0.55) (layers F.Cu F.Paste F.Mask)
+      (net 10 "Net-(C5-Pad2)"))
+    (pad 2 smd rect (at -0.5 2.75) (size 0.5 0.55) (layers F.Cu F.Paste F.Mask)
+      (net 9 "Net-(C3-Pad2)"))
+    (pad 1 smd rect (at -1.5 2.75) (size 0.5 0.55) (layers F.Cu F.Paste F.Mask)
+      (net 13 "Net-(U2-Pad1)"))
+    (pad P1 smd rect (at 0 0) (size 4.25 4.25) (layers F.Cu F.Paste F.Mask))
+  )
   (module Fiducial:Fiducial_0.5mm_Dia_1mm_Outer (layer F.Cu)
     (at 144 81)
@@
     (pad ~ smd circle (at 0 0) (size 0.5 0.5) (layers F.Cu F.Mask)
       (solder_mask_margin 0.25) (clearance 0.25))
-  )
-  (module MMA7260Q:QFN-16 (layer F.Cu)
-    (at 153.162 91.694)
-    (descr "16 LEAD QFN CASE 1622-01<br>E.g. MMA7260Q")
-    (attr smd)
-    (fp_text reference U2 (at -3.81 0) (layer F.SilkS)
-      (effects (font (size 0.801591 0.801591) (thickness 0.05)))
-    )
-    (fp_text value MMA7361L (at -0.2 -3.8) (layer F.Fab)
-      (effects (font (size 0.800764 0.800764) (thickness 0.05)))
-    )
-    (fp_line (start -3 -3) (end 3 -3) (layer Dwgs.User) (width 0.127))
-    (fp_line (start 3 -3) (end 3 3) (layer Dwgs.User) (width 0.127))
-    (fp_line (start 3 3) (end -3 3) (layer Dwgs.User) (width 0.127))
-    (fp_line (start -3 3) (end -3 -3) (layer Dwgs.User) (width 0.127))
-    (fp_line (start -2.5 -3) (end -3 -3) (layer F.SilkS) (width 0.127))
-    (fp_line (start -3 -3) (end -3 -2.5) (layer F.SilkS) (width 0.127))
-    (fp_line (start 2.5 -3) (end 3 -3) (layer F.SilkS) (width 0.127))
-    (fp_line (start 3 -3) (end 3 -2.5) (layer F.SilkS) (width 0.127))
-    (fp_line (start -3 2.5) (end -3 3) (layer F.SilkS) (width 0.127))
-    (fp_line (start -3 3) (end -2.5 3) (layer F.SilkS) (width 0.127))
-    (fp_line (start 2.5 3) (end 3 3) (layer F.SilkS) (width 0.127))
-    (fp_line (start 3 3) (end 3 2.5) (layer F.SilkS) (width 0.127))
-    (fp_circle (center -3.7 3.5) (end -3.2877 3.5) (layer F.SilkS) (width 0.1))
-    (pad P1 smd rect (at 0 0) (size 4.25 4.25) (layers F.Cu F.Paste F.Mask))
-    (pad 1 smd rect (at -1.5 2.75) (size 0.5 0.55) (layers F.Cu F.Paste F.Mask)
-      (net 13 "Net-(U2-Pad1)"))
-    (pad 2 smd rect (at -0.5 2.75) (size 0.5 0.55) (layers F.Cu F.Paste F.Mask)
-      (net 9 "Net-(C3-Pad2)"))
-    (pad 3 smd rect (at 0.5 2.75) (size 0.5 0.55) (layers F.Cu F.Paste F.Mask)
-      (net 10 "Net-(C5-Pad2)"))
-    (pad 4 smd rect (at 1.5 2.75) (size 0.5 0.55) (layers F.Cu F.Paste F.Mask)
-      (net 8 "Net-(C1-Pad2)"))
-    (pad 5 smd rect (at 2.75 1.5 90) (size 0.5 0.55) (layers F.Cu F.Paste F.Mask)
-      (net 2 GND))
-    (pad 6 smd rect (at 2.75 0.5 90) (size 0.5 0.55) (layers F.Cu F.Paste F.Mask)
-      (net 11 VCC))
-    (pad 7 smd rect (at 2.75 -0.5 90) (size 0.5 0.55) (layers F.Cu F.Paste F.Mask)
-      (net 6 "/MMA 7361 Module/Sleep"))
-    (pad 8 smd rect (at 2.75 -1.5 90) (size 0.5 0.55) (layers F.Cu F.Paste F.Mask)
-      (net 14 "Net-(U2-Pad8)"))
-    (pad 9 smd rect (at 1.5 -2.75 180) (size 0.5 0.55) (layers F.Cu F.Paste F.Mask)
-      (net 4 "/MMA 7361 Module/Og-Detect"))
-    (pad 10 smd rect (at 0.5 -2.75 180) (size 0.5 0.55) (layers F.Cu F.Paste F.Mask)
-      (net 5 "/MMA 7361 Module/g-Select"))
-    (pad 11 smd rect (at -0.5 -2.75 180) (size 0.5 0.55) (layers F.Cu F.Paste F.Mask)
-      (net 15 "Net-(U2-Pad11)"))
-    (pad 12 smd rect (at -1.5 -2.75 180) (size 0.5 0.55) (layers F.Cu F.Paste F.Mask)
-      (net 16 "Net-(U2-Pad12)"))
-    (pad 13 smd rect (at -2.75 -1.5 270) (size 0.5 0.55) (layers F.Cu F.Paste F.Mask)
-      (net 12 "/MMA 7361 Module/SelfTest"))
-    (pad 14 smd rect (at -2.75 -0.5 270) (size 0.5 0.55) (layers F.Cu F.Paste F.Mask))
-    (pad 15 smd rect (at -2.75 0.5 270) (size 0.5 0.55) (layers F.Cu F.Paste F.Mask))
-    (pad 16 smd rect (at -2.75 1.5 270) (size 0.5 0.55) (layers F.Cu F.Paste F.Mask))
   )
   (module Connector_PinHeader_1.00mm:PinHeader_1x05_P1.00mm_Vertical (layer F.Cu)
@@
     )
   )
-  (gr_text "NOTA: P1 no fue posible hallar el modelo 3d" (at 187.93 98.29) (layer Dwgs.User)
+  (dimension 22.352 (width 0.3) (layer Dwgs.User)
+    (gr_text "22,352 mm" (at 153.602 105.96) (layer Dwgs.User)
+      (effects (font (size 1.5 1.5) (thickness 0.3)))
+    )
+    (feature1 (pts (xy 164.778 98.78) (xy 164.778 104.446421)))
+    (feature2 (pts (xy 142.426 98.78) (xy 142.426 104.446421)))
+    (crossbar (pts (xy 142.426 103.86) (xy 164.778 103.86)))
+    (arrow1a (pts (xy 164.778 103.86) (xy 163.651496 104.446421)))
+    (arrow1b (pts (xy 164.778 103.86) (xy 163.651496 103.273579)))
+    (arrow2a (pts (xy 142.426 103.86) (xy 143.552504 104.446421)))
+    (arrow2b (pts (xy 142.426 103.86) (xy 143.552504 103.273579)))
+  )
+  (dimension 20.32 (width 0.3) (layer Dwgs.User)
+    (gr_text "20,320 mm" (at 171.195999 88.62 270) (layer Dwgs.User)
+      (effects (font (size 1.5 1.5) (thickness 0.3)))
+    )
+    (feature1 (pts (xy 164.778 98.78) (xy 169.68242 98.78)))
+    (feature2 (pts (xy 164.778 78.46) (xy 169.68242 78.46)))
+    (crossbar (pts (xy 169.095999 78.46) (xy 169.095999 98.78)))
+    (arrow1a (pts (xy 169.095999 98.78) (xy 168.509578 97.653496)))
+    (arrow1b (pts (xy 169.095999 98.78) (xy 169.68242 97.653496)))
+    (arrow2a (pts (xy 169.095999 78.46) (xy 168.509578 79.586504)))
+    (arrow2b (pts (xy 169.095999 78.46) (xy 169.68242 79.586504)))
+  )
+  (gr_text "NOTA: P1 no fue posible hallar el modelo 3d" (at 194.75 98.018) (layer Dwgs.User)
     (effects (font (size 1 1) (thickness 0.2)))
   )
-  (gr_text "* Componente: MMA7361\n* Pista: 0.250 mm\n* Margen: 0.25 mm\n* Mínimo ancho pista: 0.2 mm\n* Mínimo tamaño vía: 0.4 mm\n* Minimum via diameter: 1 mm\n* Terminación: HASL" (at 186.51 82.3) (layer Dwgs.User)
+  (gr_text "* Componente: MMA7361\n* Pista: 0.250 mm\n* Margen: 0.25 mm\n* Mínimo ancho pista: 0.2 mm\n* Mínimo tamaño vía: 0.4 mm\n* Minimum via diameter: 1 mm\n* Terminación: HASL" (at 189.924 83.54) (layer Dwgs.User)
     (effects (font (size 1 1) (thickness 0.2)))
   )
