File: MMA7361/MMA7361.sch (KiCad schematic (older format))
At the start: 0 parts

Commit message: More changes
Parts:
- added MH? (x4): MountingHole, symbol Mechanical:MountingHole
Changed lines of the file:
@@
 F1 "acel.sch" 50
 $EndSheet
+$Comp
+L Mechanical:MountingHole MH?
+U 1 1 5BD31F88
+P 5600 5150
+F 0 "MH?" H 5700 5196 50  0000 L CNN
+F 1 "MountingHole" H 5700 5105 50  0000 L CNN
+F 2 "" H 5600 5150 50  0001 C CNN
+F 3 "~" H 5600 5150 50  0001 C CNN
+	1    5600 5150
+	1    0    0    -1
+$EndComp
+$Comp
+L Mechanical:MountingHole MH?
+U 1 1 5BD3205B
+P 6550 5150
+F 0 "MH?" H 6650 5196 50  0000 L CNN
+F 1 "MountingHole" H 6650 5105 50  0000 L CNN
+F 2 "" H 6550 5150 50  0001 C CNN
+F 3 "~" H 6550 5150 50  0001 C CNN
+	1    6550 5150
+	1    0    0    -1
+$EndComp
+$Comp
+L Mechanical:MountingHole MH?
+U 1 1 5BD320E3
+P 5600 5650
+F 0 "MH?" H 5700 5696 50  0000 L CNN
+F 1 "MountingHole" H 5700 5605 50  0000 L CNN
+F 2 "" H 5600 5650 50  0001 C CNN
+F 3 "~" H 5600 5650 50  0001 C CNN
+	1    5600 5650
+	1    0    0    -1
+$EndComp
+$Comp
+L Mechanical:MountingHole MH?
+U 1 1 5BD32158
+P 6550 5650
+F 0 "MH?" H 6650 5696 50  0000 L CNN
+F 1 "MountingHole" H 6650 5605 50  0000 L CNN
+F 2 "" H 6550 5650 50  0001 C CNN
+F 3 "~" H 6550 5650 50  0001 C CNN
+	1    6550 5650
+	1    0    0    -1
+$EndComp
 $EndSCHEMATC

Commit message: The last change have been added
Parts:
- removed MH? (x4): MountingHole, symbol Mechanical:MountingHole
Changed lines of the file:
@@
 Date ""
 Rev ""
-Comp "CESE"
+Comp "Diseño de circuitos impresos"
 Comment1 ""
 Comment2 ""
@@
 F1 "acel.sch" 50
 $EndSheet
-$Comp
-L Mechanical:MountingHole MH?
-U 1 1 5BD31F88
-P 5600 5150
-F 0 "MH?" H 5700 5196 50  0000 L CNN
-F 1 "MountingHole" H 5700 5105 50  0000 L CNN
-F 2 "" H 5600 5150 50  0001 C CNN
-F 3 "~" H 5600 5150 50  0001 C CNN
-	1    5600 5150
-	1    0    0    -1
-$EndComp
-$Comp
-L Mechanical:MountingHole MH?
-U 1 1 5BD3205B
-P 6550 5150
-F 0 "MH?" H 6650 5196 50  0000 L CNN
-F 1 "MountingHole" H 6650 5105 50  0000 L CNN
-F 2 "" H 6550 5150 50  0001 C CNN
-F 3 "~" H 6550 5150 50  0001 C CNN
-	1    6550 5150
-	1    0    0    -1
-$EndComp
-$Comp
-L Mechanical:MountingHole MH?
-U 1 1 5BD320E3
-P 5600 5650
-F 0 "MH?" H 5700 5696 50  0000 L CNN
-F 1 "MountingHole" H 5700 5605 50  0000 L CNN
-F 2 "" H 5600 5650 50  0001 C CNN
-F 3 "~" H 5600 5650 50  0001 C CNN
-	1    5600 5650
-	1    0    0    -1
-$EndComp
-$Comp
-L Mechanical:MountingHole MH?
-U 1 1 5BD32158
-P 6550 5650
-F 0 "MH?" H 6650 5696 50  0000 L CNN
-F 1 "MountingHole" H 6650 5605 50  0000 L CNN
-F 2 "" H 6550 5650 50  0001 C CNN
-F 3 "~" H 6550 5650 50  0001 C CNN
-	1    6550 5650
-	1    0    0    -1
-$EndComp
 $EndSCHEMATC

Commit message: The last version have been added
Parts:
- added C1, C3: 1 µF, Footprints:C_0805_2012Metric_Pad1.15x1.40mm_HandSolder, symbol MMA7361-rescue:CP1-Device
- added C2, C4: 470 µF, Footprints:C_0805_2012Metric_Pad1.15x1.40mm_HandSolder, symbol MMA7361-rescue:C-Device
- added C5, C6, C7: 3.3nf, Footprints:C_0805_2012Metric_Pad1.15x1.40mm_HandSolder, symbol MMA7361-rescue:C-Device
- added D1: LED, Footprints:LED_0805_2012Metric_Pad1.15x1.40mm_HandSolder, symbol MMA7361-rescue:LED-Device
- added F1, F2, F3: Fiducial, Footprints:Fiducial_1mm_Dia_2mm_Outer, symbol MMA7361-rescue:MountingHole-Mechanical
- added J1, J2: Conn_01x05, Footprints:PinHeader_1x05_P2.54mm_Vertical, symbol MMA7361-rescue:Conn_01x05-Connector_Generic
- added R1: 1 K, Footprints:R_0805_2012Metric_Pad1.15x1.40mm_HandSolder, symbol MMA7361-rescue:R-Device
- added U1: RT9161, Footprints:SOT-89-3_Handsoldering, symbol MMA7361:RT9601
- added U2: MMA7361L, Footprints:LGA-14_3x5mm_P0.8mm_LayoutBorder1x6y, symbol MMA7361:MMA7361L
Connections:
- net labels added: +5V, GND, Og-Detect, SelfTest, VCC, X, Y, Z, g-Select, ~Sleep
- wire segments 0 -> 60
Other:
- note added: "Fiducial"
- note added: "U1 RT9161"
- note added: "U2 MMA7361L"
